File: hardware/led-strip-v2.kicad_sch (KiCad schematic)
At the start: 41 parts

Commit message: Data Cleanup
Parts:
- C1: value (none) -> 220pF; footprint (none) -> kicad-libraries:C0402F
- C2: value (none) -> 10uF; footprint (none) -> kicad-libraries:C0805E
- C3, C4, C5, C8, C9: value (none) -> 100nF; footprint (none) -> kicad-libraries:C0603F
- C6, C7: value (none) -> DNP; footprint (none) -> kicad-libraries:C0603F
- D1, D2: value (none) -> ESD5V0D3B-TP; footprint (none) -> kicad-libraries:SOD-323
- D3: value (none) -> blue; footprint (none) -> kicad-libraries:D0603F
- J1, J2, J3: value (none) -> AKL_5_2; footprint (none) -> kicad-libraries:AKL_5_2
- L1: value (none) -> 0; footprint (none) -> kicad-libraries:R0603F
- L2: value (none) -> FB; footprint (none) -> kicad-libraries:R0603F
- P1: value (none) -> CON-SENSOR; footprint (none) -> kicad-libraries:CON-SENSOR2
- P2, P3, P4, P5, P6, P7: value (none) -> TST; footprint (none) -> kicad-libraries:SOLDER_PAD2
- P8: value (none) -> Boot; footprint (none) -> kicad-libraries:SolderJumper
- P9: value (none) -> Debug; footprint (none) -> kicad-libraries:DEBUG_PAD
- R1, R3: value (none) -> 1k; footprint (none) -> kicad-libraries:R0603F
- R2: value (none) -> 10k; footprint (none) -> kicad-libraries:R0603F
- R4, R5: value (none) -> 470; footprint (none) -> kicad-libraries:R0603F
- R6, R7: value (none) -> 100; footprint (none) -> kicad-libraries:R0603F
- RP1: value (none) -> 82; footprint (none) -> kicad-libraries:4X0402
- U1: value (none) -> XMC1302; footprint (none) -> kicad-libraries:QFN24-4x4mm-0.5mm
- U2, U3, U4, U5: value (none) -> DRILL; footprint (none) -> kicad-libraries:DRILL_NP
- U6, U7: value (none) -> 74LVC1G17; footprint (none) -> kicad-libraries:SOT23-5
Other:
- note added: "Copyright Tinkerforge GmbH 2023. This documentation describes Open Hardware and is licensed under the CERN OHL v. 1.1. You may redistribute and modify this documentation under the terms of the CERN OHL v.1.1. (http://ohwr.org/cernohl). This documentation is distributed WITHOUT ANY EXPRESS OR IMPLIED WARRANTY, INCLUDING OF MERCHANTABILITY, SATISFACTORY QUALITY AND FITNESS FOR A PARTICULAR PURPOSE.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"
- note removed: "Copyright Tinkerforge GmbH 2018. This documentation describes Open Hardware and is licensed under the CERN OHL v. 1.1. You may redistribute and modify this documentation under the terms of the CERN OHL v.1.1. (http://ohwr.org/cernohl). This documentation is distributed WITHOUT ANY EXPRESS OR IMPLIED WARRANTY, INCLUDING OF MERCHANTABILITY, SATISFACTORY QUALITY AND FITNESS FOR A PARTICULAR PURPOSE.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"

Commit message: update to kicad 7. updated schematic version v2.2 detection. updatet schematic pdf
Connections:
- net GND: now also U1.8 (P2.11_AIO)
- no-connect marks 12 -> 11
Other:
- note added: "Version Detection V2.2"
- moved on the sheet: P9
